File: MyProSole.kicad_sch (KiCad schematic)
At the start: 2 parts, among them J1 Conn_01x07_Socket_XIAO_ESP32C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, J2 Conn_01x07_Socket_XIAO_ESP32C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

Commit message: Schaltplan Teil 1 fertig
Parts:
- added C1, C2, C3: 100nF, symbol Device:C_Small
- added D1: WS2812B, LED_SMD:LED_WS2812B_PLCC4_5.0x5.0mm_P3.2mm, symbol LED:WS2812B
- added J3: i2c-bus, symbol Connector_Generic:Conn_01x04
- added J4: FSR1, symbol Connector_Generic:Conn_01x02
- added J5: FSR2, symbol Connector_Generic:Conn_01x02
- added J6: FSR3, symbol Connector_Generic:Conn_01x02
- added J7: Conn_01x06, symbol Connector_Generic:Conn_01x06
- added R1, R2, R3: 2kΩ, symbol Device:R_Small
- added TP1: TestPoint, symbol Connector:TestPoint
- J2: value Conn_01x07_Socket_XIAO_ESP32C3_Right -> XIAO_ESP32C3
Connections:
- net CS: now reaches J2.1 (GPIO_20)
- net CS: now also J7.6 (Pin_6)
- net SCK: now reaches J2.2 (GPIO_8)
- net SCK: now also J7.5 (Pin_5)
- net MISO: now reaches J2.3 (GPIO_9)
- net MISO: now also J7.4 (Pin_4)
- net MOSI: now reaches J2.4 (GPIO_10)
- net MOSI: now also J7.3 (Pin_3)
- net +3.3V: now reaches J2.5 (3V3)
- net +3.3V: now also J3.1 (Pin_1), J4.1 (Pin_1), J5.1 (Pin_1), J6.1 (Pin_1), J7.1 (Pin_1)
- net GND: now reaches J2.6 (GND)
- net GND: now also C1.1, C2.1, C3.1, D1.3 (VSS), J3.4 (Pin_4), J7.2 (Pin_2), R1.1, R2.1, R3.1
- net +5V: now reaches J2.7 (5V)
- net +5V: now also D1.1 (VDD)
- net FSR1_ADC: now reaches J1.1 (GPIO_2)
- net FSR1_ADC: now also C1.2, J6.2 (Pin_2), R1.2
- net FSR2_ADC: now reaches J1.2 (GPIO_3)
- net FSR2_ADC: now also C2.2, J5.2 (Pin_2), R2.2
- net FSR3_ADC: now reaches J1.3 (GPIO_5)
- net FSR3_ADC: now also C3.2, J4.2 (Pin_2), R3.2
- net RGB_LED: now reaches J1.4 (GPIO_5)
- net RGB_LED: now also D1.4 (DIN)
- net SDA: now reaches J1.5 (GPIO_6)
- net SDA: now also J3.3 (Pin_3)
- net SCL: now reaches J1.6 (GPIO_7)
- net SCL: now also J3.2 (Pin_2)
- net at J1.7 (GPIO_21): now also TP1.1
Other:
- moved on the sheet: J1
